File: routage/Analogique_A2S1/CarteAnalogique_V1_0/CarteAnalogique_V1_0.kicad_sch (KiCad schematic)
At the start: 8 parts, among them J1 Barrel_Jack, U1 LM7805_TO220, U2 MCP602, U3 LM35-LP

Commit message: Creation du routage
Parts:
- added C3: 150pF, Capacitor_THT:C_Axial_L5.1mm_D3.1mm_P10.00mm_Horizontal, symbol Device:C
- added D1: DIODE, Diode_THT:D_A-405_P12.70mm_Horizontal, symbol pspice:DIODE
- added D2: LED, LED_THT:LED_D8.0mm, symbol Device:LED
- added R3, R4: 10K, Resistor_THT:R_Axial_DIN0411_L9.9mm_D3.6mm_P7.62mm_Vertical, symbol Device:R
- added SW1: SW_Push_Dual_x2, Button_Switch_THT:SW_PUSH_6mm_H13mm, symbol Switch:SW_Push_Dual_x2
- added U4: ADC0801LCN, lib:DIP254P762X508-20, symbol ADC0801LCN:ADC0801LCN
- added U5: AT28C64B-15PU, lib:EEPROM, symbol AT28C64B-15PU:AT28C64B-15PU
- added U6, U7: TIL311, lib:TIL311, symbol TIL311:TIL311
- C1: footprint Capacitor_THT:CP_Axial_L18.0mm_D8.0mm_P25.00mm_Horizontal -> Capacitor_THT:CP_Radial_D7.5mm_P2.50mm
- C2: footprint Capacitor_THT:CP_Axial_L18.0mm_D8.0mm_P25.00mm_Horizontal -> Capacitor_THT:CP_Radial_D8.0mm_P3.80mm
- J1: footprint Connector_BarrelJack:BarrelJack_CLIFF_FC681465S_SMT_Horizontal -> Connector_BarrelJack:BarrelJack_CUI_PJ-063AH_Horizontal
- R1, R2: footprint Resistor_THT:R_Axial_DIN0918_L18.0mm_D9.0mm_P25.40mm_Horizontal -> Resistor_THT:R_Axial_DIN0411_L9.9mm_D3.6mm_P7.62mm_Vertical
- U2: footprint (none) -> Package_DIP:DIP-8_W10.16mm
Connections:
- net +5V: now also R4.1, U4.20 (VCC), U5.28 (VCC), U6.1 (LED_SUPPLY), U6.14 (LOGIC_SUPPLY), U7.1 (LED_SUPPLY), U7.14 (LOGIC_SUPPLY)
- net GND: now also C3.2, D2.1 (K), SW1.2 (D), U4.1 (~CS), U4.10 (DGND), U4.2 (~RD), U4.7 (VIN-), U4.8 (AGND), U5.14 (GND), U5.2 (A12), U5.20 (~{CE}), U5.21 (A10), U5.22 (~{OE}), U5.23 (A11), U5.24 (A9), U5.25 (A8), U5.27 (~{WE}), U6.10 (RIGHT_DECIMAL_), U6.4 (LEFT_DECIMAL), U6.5 (STROBE_INPUT), U6.7 (GROUND), U6.8 (BLANKING_INPUT), U7.10 (RIGHT_DECIMAL_), U7.4 (LEFT_DECIMAL), U7.5 (STROBE_INPUT), U7.7 (GROUND), U7.8 (BLANKING_INPUT)
- net Vcapteur: now also U4.6 (VIN+)
- net +12V: no longer names the net of C1.1, U1.1 (VI)
- net +12V: now also D1.2 (A); no longer J1.1
- new net: D2.2 (A), R4.2
- new net: D1.1 (K), J1.1
- new net: R3.1, U4.19 (CLKR)
- new net: C3.1, R3.2, U4.4 (CLKIN)
- new net: U4.18 (DB0), U5.10 (A0)
- new net: U4.11 (DB7), U5.3 (A7)
- new net: U4.12 (DB6), U5.4 (A6)
- new net: U4.13 (DB5), U5.5 (A5)
- new net: U4.14 (DB4), U5.6 (A4)
- new net: U4.15 (DB3), U5.7 (A3)
- new net: U4.16 (DB2), U5.8 (A2)
- new net: U4.17 (DB1), U5.9 (A1)
- new net: SW1.1 (C), U4.3 (~WR), U4.5 (~INTR)
- new net B0: U5.11 (I/O0), U6.3 (DATA_INPUT_A)
- new net B1: U5.12 (I/O1), U6.2 (DATA_INPUT_B)
- new net B2: U5.13 (I/O2), U6.12 (DATA_INPUT_D)
- new net B3: U5.15 (I/O3), U6.13 (DATA_INPUT_C)
- new net B4: U5.16 (I/O4), U7.3 (DATA_INPUT_A)
- new net B5: U5.17 (I/O5), U7.2 (DATA_INPUT_B)
- new net B6: U5.18 (I/O6), U7.13 (DATA_INPUT_C)
- new net B7: U5.19 (I/O7), U7.12 (DATA_INPUT_D)
Other:
- moved on the sheet: C1, C2, J1, R1, R2, U1, U2A, U2C, U3

Commit message: routage du projet Analogique premier semestre fermeture de la branche et merge
Parts:
- C2: value 0,33 uF -> 0,1 uF
- R1: value 90K -> 56K
- R4: value 10K -> 300
Changed lines of the file:
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@@
     (in_bom yes) (on_board yes)
     (property "Reference" "R4" (id 0) (at 91.44 71.12 0))
-    (property "Value" "10K" (id 1) (at 91.44 73.66 0))
+    (property "Value" "300" (id 1) (at 91.44 73.66 0))
     (property "Footprint" "Resistor_THT:R_Axial_DIN0411_L9.9mm_D3.6mm_P7.62mm_Vertical" (id 2) (at 84.582 73.66 90)
       (effects (font (size 1.27 1.27)) hide)
@@
     (in_bom yes) (on_board yes)
     (property "Reference" "R1" (id 0) (at 80.01 121.92 90))
-    (property "Value" "90K" (id 1) (at 80.01 127 90))
+    (property "Value" "56K" (id 1) (at 80.01 127 90))
     (property "Footprint" "Resistor_THT:R_Axial_DIN0411_L9.9mm_D3.6mm_P7.62mm_Vertical" (id 2) (at 80.01 122.682 90)
       (effects (font (size 1.27 1.27)) hide)
@@
       (effects (font (size 1.27 1.27)) (justify left))
     )
-    (property "Value" "0,33 uF" (id 1) (at 77.47 75.5649 0)
+    (property "Value" "0,1 uF" (id 1) (at 77.47 75.5649 0)
       (effects (font (size 1.27 1.27)) (justify left))
     )
@@
     )
     (path "/ee4ac81e-dd78-4726-8d1a-360f968b384e"
-      (reference "C2") (unit 1) (value "0,33 uF") (footprint "Capacitor_THT:CP_Radial_D8.0mm_P3.80mm")
+      (reference "C2") (unit 1) (value "0,1 uF") (footprint "Capacitor_THT:CP_Radial_D8.0mm_P3.80mm")
     )
     (path "/8e275fbd-6e21-457e-bf18-619dfbde4912"
@@
     )
     (path "/78815e58-e1b1-4dcd-bc4b-68a5fcf24390"
-      (reference "R1") (unit 1) (value "90K") (footprint "Resistor_THT:R_Axial_DIN0411_L9.9mm_D3.6mm_P7.62mm_Vertical")
+      (reference "R1") (unit 1) (value "56K") (footprint "Resistor_THT:R_Axial_DIN0411_L9.9mm_D3.6mm_P7.62mm_Vertical")
     )
     (path "/1b6f430b-1b32-4822-9df7-17ce1e0949ed"
@@
     )
     (path "/65ec78cc-6a9e-49fe-9f5f-bed4423daff9"
-      (reference "R4") (unit 1) (value "10K") (footprint "Resistor_THT:R_Axial_DIN0411_L9.9mm_D3.6mm_P7.62mm_Vertical")
+      (reference "R4") (unit 1) (value "300") (footprint "Resistor_THT:R_Axial_DIN0411_L9.9mm_D3.6mm_P7.62mm_Vertical")
     )
     (path "/f8a57dc6-fc37-44cd-a471-98c4d01557da"
