File: routage/Numerique_A2S2/testLCD.kicad_sch (KiCad schematic)
At the start: 15 parts, among them J3 Barrel_Jack, J4 Conn_01x06_Pin, SW2 SW_Push, U3 LM7805_TO220, U4 PIC16F876-XXISO, Y2 Crystal

Commit message: Modification condo
Parts:
- C7: value C -> 10p
- C8: value ~ -> 10p
